File: led_display_digit.kicad_sch (KiCad schematic)
At the start: 118 parts, among them J1 Conn_01x05, J2 Conn_01x07, Q1 2N7002, Q2 2N7002, Q3 2N7002, Q4 2N7002

Commit message: little design changes
Parts:
- added H1, H2: MHole, MountingHole:MountingHole_2.2mm_M2_Pad, symbol Mechanical:MountingHole_Pad
Connections:
- net GND: now also H1.1, H2.1
Other:
- moved on the sheet: J1
